File: elec/layout/default/default.kicad_pcb (KiCad board)
At the start: 4 copper layers, 0 parts

Commit message: layout: save imported and placed board
Parts:
- added BT1: ?, Connector_JST:JST_PH_B2B-PH-K_1x02_P2.00mm_Vertical, F.Cu at (-29.2, -22.4)
- added C1: ?, Capacitor_SMD:C_0603_1608Metric, F.Cu at (0.32, -104.3)
- added C10: ?, Capacitor_SMD:C_0603_1608Metric, F.Cu at (0.32, -99.8)
- added C11: ?, Capacitor_SMD:C_0603_1608Metric, F.Cu at (-36.3, -19.3)
- added C12: ?, Capacitor_SMD:C_0603_1608Metric, F.Cu at (0.32, -108.8)
- added C13: ?, Capacitor_SMD:C_0603_1608Metric, F.Cu at (-36.3, -23.8)
- added C14: ?, Capacitor_SMD:C_0603_1608Metric, F.Cu at (-63.3, -21.1)
- added C15: ?, Capacitor_SMD:C_0603_1608Metric, F.Cu at (0.32, -95.3)
- added C16: ?, Capacitor_SMD:C_0603_1608Metric, F.Cu at (-48.9, -17.8)
- added C17: ?, Capacitor_SMD:C_0603_1608Metric, F.Cu at (0.32, -90.8)
- added C18: ?, Capacitor_SMD:C_0603_1608Metric, F.Cu at (-69.3, -21.1)
- added C19: ?, Capacitor_SMD:C_0603_1608Metric, F.Cu at (6.23, -47.9)
- added C2: ?, Capacitor_SMD:C_0805_2012Metric, F.Cu at (-0.00, -47.7)
- added C20: ?, Capacitor_SMD:C_0805_2012Metric, F.Cu at (-1.52, -40.3)
- added C21: ?, Capacitor_SMD:C_0603_1608Metric, F.Cu at (-55.2, -18.1)
- added C22: ?, Capacitor_SMD:C_0402_1005Metric, F.Cu at (-69.9, -16.9)
- added C3: ?, Capacitor_SMD:C_0805_2012Metric, F.Cu at (4.89, -34.9)
- added C4: ?, Capacitor_SMD:C_0805_2012Metric, F.Cu at (-1.56, -34.9)
- added C5: ?, Capacitor_SMD:C_0402_1005Metric, F.Cu at (-9.42, -91.6)
- added C6: ?, Capacitor_SMD:C_0402_1005Metric, F.Cu at (-9.42, -95.5)
- added C7: ?, Capacitor_SMD:C_0402_1005Metric, F.Cu at (-14.3, -91.6)
- added C8: ?, Capacitor_SMD:C_0805_2012Metric, F.Cu at (4.93, -40.3)
- added C9: ?, Capacitor_SMD:C_0402_1005Metric, F.Cu at (-63.8, -16.9)
- added D1: ?, Diode_SMD:D_SOD-123, F.Cu at (-16.7, -27.2)
- added D2: ?, Diode_SMD:D_SOD-123, F.Cu at (-16.7, -21.9)
- added D3: ?, Diode_SMD:D_SOD-123, F.Cu at (-8.62, -40.1)
- added D4: ?, hp42s:Vishay_VSMB2943SLX01_SideView, F.Cu at (-448.9, -462.5)
- added D5: ?, hp42s:Dialight_599_BiColor_1208_RA, F.Cu at (-422.9, -462.3)
- added D6: ?, Diode_SMD:D_SOD-123, F.Cu at (-16.7, -32.6)
- added J1: ?, Connector_USB:USB_C_Receptacle_GCT_USB4105-xx-A_16P_TopMnt_Horizontal, F.Cu at (-434.9, -460.5)
- added J2: ?, Connector_FFC-FPC:Hirose_FH12-24S-0.5SH_1x24-1MP_P0.50mm_Horizontal, B.Cu at (-461.9, -434.0)
- added L1: ?, Inductor_SMD:L_Coilcraft_XxL4020, F.Cu at (-8.75, -27.2)
- added L2: ?, Inductor_SMD:L_Bourns-SRN4018, F.Cu at (-16.6, -39.0)
- added L3: ?, Inductor_SMD:L_APV_ANR3015, F.Cu at (5.51, -27.7)
- added LS1: ?, Buzzer_Beeper:Buzzer_Murata_PKLCS1212E, F.Cu at (-44.0, -105.9)
- added Q1: ?, Package_TO_SOT_SMD:SOT-323_SC-70, F.Cu at (6.30, -90.3)
- added Q2: ?, Package_TO_SOT_SMD:SOT-23, F.Cu at (5.54, -21.1)
- added R1: ?, Resistor_SMD:R_0402_1005Metric, F.Cu at (5.78, -100.1)
- added R10: ?, Resistor_SMD:R_0402_1005Metric, F.Cu at (6.85, -60.2)
- added R11: ?, Resistor_SMD:R_0402_1005Metric, F.Cu at (-44.0, -96.1)
- added R12: ?, Resistor_SMD:R_0402_1005Metric, F.Cu at (-39.1, -92.1)
- added R13: ?, Resistor_SMD:R_0402_1005Metric, F.Cu at (6.85, -80.3)
- added R14: ?, Resistor_SMD:R_0402_1005Metric, F.Cu at (6.85, -52.3)
- added R15: ?, Resistor_SMD:R_0402_1005Metric, F.Cu at (6.85, -56.2)
- added R16: ?, Resistor_SMD:R_0402_1005Metric, F.Cu at (-34.2, -92.1)
- added R17: ?, Resistor_SMD:R_0402_1005Metric, F.Cu at (5.78, -104.6)
- added R18: ?, Resistor_SMD:R_0402_1005Metric, F.Cu at (5.78, -109.1)
- added R19: ?, Resistor_SMD:R_0402_1005Metric, F.Cu at (-34.2, -96.1)
- added R2: ?, Resistor_SMD:R_0402_1005Metric, F.Cu at (-18.2, -17.2)
- added R20: ?, Resistor_SMD:R_0402_1005Metric, F.Cu at (6.85, -68.3)
- added R21: ?, Resistor_SMD:R_0402_1005Metric, F.Cu at (-14.3, -95.5)
- added R22: ?, Resistor_SMD:R_0402_1005Metric, F.Cu at (6.85, -84.3)
- added R23: ?, Resistor_SMD:R_0402_1005Metric, F.Cu at (-33.6, -103.7)
- added R24: ?, Resistor_SMD:R_0402_1005Metric, F.Cu at (-44.0, -92.1)
- added R3: ?, Resistor_SMD:R_0402_1005Metric, F.Cu at (-33.6, -107.7)
- added R4: ?, Resistor_SMD:R_0402_1005Metric, F.Cu at (5.78, -95.6)
- added R5: ?, Resistor_SMD:R_0402_1005Metric, F.Cu at (6.85, -76.4)
- added R6: ?, Resistor_SMD:R_0402_1005Metric, F.Cu at (-39.1, -96.1)
- added R7: ?, Resistor_SMD:R_0402_1005Metric, F.Cu at (6.85, -64.3)
- added R8: ?, Resistor_SMD:R_0402_1005Metric, F.Cu at (-33.6, -111.7)
- added R9: ?, Resistor_SMD:R_0402_1005Metric, F.Cu at (6.85, -72.3)
- added SW1: ?, hp42s:Dome_4Leg_8.5mm, F.Cu at (-464.2, -402.1)
- added SW10: ?, hp42s:Dome_4Leg_8.5mm, F.Cu at (-426.7, -390.1)
- added SW11: ?, hp42s:Dome_4Leg_8.5mm, F.Cu at (-414.2, -390.1)
- added SW12: ?, hp42s:Dome_4Leg_8.5mm, F.Cu at (-401.7, -390.1)
- added SW13: ?, hp42s:Dome_4Leg_8.5mm, F.Cu at (-464.2, -378.1)
- added SW14: ?, hp42s:Dome_4Leg_8.5mm, F.Cu at (-439.2, -378.1)
- added SW15: ?, hp42s:Dome_4Leg_8.5mm, F.Cu at (-426.7, -378.1)
- added SW16: ?, hp42s:Dome_4Leg_8.5mm, F.Cu at (-414.2, -378.1)
- added SW17: ?, hp42s:Dome_4Leg_8.5mm, F.Cu at (-401.7, -378.1)
- added SW18: ?, hp42s:Dome_4Leg_8.5mm, F.Cu at (-464.2, -366.1)
- added SW19: ?, hp42s:Dome_4Leg_10mm, F.Cu at (-447.9, -366.1)
- added SW2: ?, hp42s:Dome_4Leg_8.5mm, F.Cu at (-451.7, -402.1)
- added SW20: ?, hp42s:Dome_4Leg_10mm, F.Cu at (-432.9, -366.1)
- added SW21: ?, hp42s:Dome_4Leg_10mm, F.Cu at (-417.9, -366.1)
- added SW22: ?, hp42s:Dome_4Leg_10mm, F.Cu at (-402.9, -366.1)
- added SW23: ?, hp42s:Dome_4Leg_8.5mm, F.Cu at (-464.2, -354.1)
- added SW24: ?, hp42s:Dome_4Leg_10mm, F.Cu at (-447.9, -354.1)
- added SW25: ?, hp42s:Dome_4Leg_10mm, F.Cu at (-432.9, -354.1)
- added SW26: ?, hp42s:Dome_4Leg_10mm, F.Cu at (-417.9, -354.1)
- added SW27: ?, hp42s:Dome_4Leg_10mm, F.Cu at (-402.9, -354.1)
- added SW28: ?, hp42s:Dome_4Leg_8.5mm, F.Cu at (-464.2, -342.1)
- added SW29: ?, hp42s:Dome_4Leg_10mm, F.Cu at (-447.9, -342.1)
- added SW3: ?, hp42s:Dome_4Leg_8.5mm, F.Cu at (-439.2, -402.1)
- added SW30: ?, hp42s:Dome_4Leg_10mm, F.Cu at (-432.9, -342.1)
- added SW31: ?, hp42s:Dome_4Leg_10mm, F.Cu at (-417.9, -342.1)
- added SW32: ?, hp42s:Dome_4Leg_10mm, F.Cu at (-402.9, -342.1)
- added SW33: ?, hp42s:Dome_4Leg_8.5mm, F.Cu at (-464.2, -330.1)
- added SW34: ?, hp42s:Dome_4Leg_10mm, F.Cu at (-447.9, -330.1)
- added SW35: ?, hp42s:Dome_4Leg_10mm, F.Cu at (-432.9, -330.1)
- added SW36: ?, hp42s:Dome_4Leg_10mm, F.Cu at (-417.9, -330.1)
- added SW37: ?, hp42s:Dome_4Leg_10mm, F.Cu at (-402.9, -330.1)
- added SW38: ?, hp42s:Dome_4Leg_8.5mm, F.Cu at (-451.7, -378.1)
- added SW39: ?, Button_Switch_SMD:SW_SPDT_CK_JS102011SAQN, F.Cu at (-459.9, -461.1)
- added SW4: ?, hp42s:Dome_4Leg_8.5mm, F.Cu at (-426.7, -402.1)
- added SW40: ?, hp42s:Alps_SKRTLAE010_SidePush, F.Cu at (-404.9, -462.6)
- added SW41: ?, hp42s:Alps_SKRTLAE010_SidePush, F.Cu at (-413.9, -462.6)
- added SW5: ?, hp42s:Dome_4Leg_8.5mm, F.Cu at (-414.2, -402.1)
- added SW6: ?, hp42s:Dome_4Leg_8.5mm, F.Cu at (-401.7, -402.1)
- added SW7: ?, hp42s:Dome_4Leg_8.5mm, F.Cu at (-464.2, -390.1)
- added SW8: ?, hp42s:Dome_4Leg_8.5mm, F.Cu at (-451.7, -390.1)
- added SW9: ?, hp42s:Dome_4Leg_8.5mm, F.Cu at (-439.2, -390.1)
- added TP1: ?, TestPoint:TestPoint_Pad_D1.5mm, F.Cu at (-28.1, -94.8)
- added TP10: ?, TestPoint:TestPoint_Pad_D1.5mm, F.Cu at (-22.5, -94.8)
- added TP11: ?, TestPoint:TestPoint_Pad_D1.5mm, F.Cu at (0.09, -121.9)
- added TP2: ?, TestPoint:TestPoint_Pad_D1.5mm, F.Cu at (5.64, -116.3)
- added TP3: ?, TestPoint:TestPoint_Pad_3.0x3.0mm, F.Cu at (-1.44, -20.8)
- added TP4: ?, TestPoint:TestPoint_Pad_D1.5mm, F.Cu at (-49.2, -95.4)
- added TP5: ?, TestPoint:TestPoint_Pad_D1.5mm, F.Cu at (-49.2, -89.8)
- added TP6: ?, TestPoint:TestPoint_Pad_D1.5mm, F.Cu at (-28.1, -89.2)
- added TP7: ?, TestPoint:TestPoint_Pad_D1.5mm, F.Cu at (5.64, -121.9)
- added TP8: ?, TestPoint:TestPoint_Pad_D1.5mm, F.Cu at (0.09, -116.3)
- added TP9: ?, TestPoint:TestPoint_Pad_D1.5mm, F.Cu at (-22.5, -89.2)
- added U1: ?, hp42s:TI_DQA0010A_USON-10_2.5x1mm_P0.5mm, F.Cu at (-42.4, -23.4)
- added U2: ?, Package_DFN_QFN:Texas_DSQ0010A_WSON-10-1EP_2x2mm_P0.4mm_EP0.9x1.5mm, F.Cu at (-55.1, -23.2)
- added U3: ?, hp42s:TI_DSK0010A_WSON-10-1EP_2.5x2.5mm_P0.5mm_EP2x1.2mm, F.Cu at (-48.7, -23.1)
- added U4: ?, Package_DFN_QFN:TDFN-8-1EP_2x2mm_P0.5mm_EP0.8x1.2mm, F.Cu at (-42.5, -17.9)
- added U5: ?, RF_Module:ESP32-S2-MINI-1, F.Cu at (-76.2, -98.4)
- added U6: ?, Package_TO_SOT_SMD:SOT-23-6, F.Cu at (-1.39, -27.6)
Other:
- board outline added: 76 x 144 mm

Commit message: layout: save imported and placed board
Parts:
- moved D5 63.2 mm to (-366.5, -490.7)
- moved J1 63.2 mm to (-378.5, -488.8)
- moved J2 63.2 mm to (-405.5, -462.4)
- moved R18 63.2 mm to (62.2, -137.5)
- moved R20 63.2 mm to (63.3, -96.7)
- moved R8 63.2 mm to (22.9, -140.1)
- moved SW1 63.2 mm to (-407.8, -430.5)
- moved SW10 63.2 mm to (-370.2, -418.5)
- moved SW11 63.2 mm to (-357.8, -418.5)
- moved SW12 63.2 mm to (-345.2, -418.5)
- moved SW13 63.2 mm to (-407.8, -406.5)
- moved SW14 63.2 mm to (-382.8, -406.5)
- moved SW15 63.2 mm to (-370.2, -406.5)
- moved SW16 63.2 mm to (-357.8, -406.5)
- moved SW17 63.2 mm to (-345.2, -406.5)
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
Commit message: layout: save imported and placed board
Parts:
- moved BT1 775.4 mm to (-515.7, -604.2)
- moved C1 775.4 mm to (-486.2, -686.2)
- moved C10 775.4 mm to (-486.2, -681.7)
- moved C11 775.4 mm to (-522.9, -601.2)
- moved C12 775.4 mm to (-486.2, -690.7)
- moved C13 775.4 mm to (-522.9, -605.7)
- moved C14 775.4 mm to (-549.8, -603.0)
- moved C15 775.4 mm to (-486.2, -677.2)
- moved C16 775.4 mm to (-535.4, -599.6)
- moved C17 775.4 mm to (-486.2, -672.7)
- moved C18 775.4 mm to (-555.8, -603.0)
- moved C19 775.4 mm to (-480.3, -629.8)
- moved C2 775.4 mm to (-486.6, -629.5)
- moved C20 775.4 mm to (-488.1, -622.1)
- moved C21 775.4 mm to (-541.8, -600.0)
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