File: elec/layout/default/default.kicad_pcb (KiCad board)
At the start: 4 copper layers, 76 x 144 mm, 119 parts, among them J1 ?, J2 ?, Q1 ?, Q2 ?, SW1 ?, SW10 ?, SW11 ?, SW12 ?, SW13 ?, SW14 ?, SW15 ?, SW16 ?, SW17 ?, SW18 ?, SW19 ?, SW2 ?, SW20 ?, SW21 ?, SW22 ?, SW23 ?, SW24 ?, SW25 ?, SW26 ?, SW27 ?, SW28 ?, SW29 ?, SW3 ?, SW30 ?, SW31 ?, SW32 ?, SW33 ?, SW34 ?, SW35 ?, SW36 ?, SW37 ?, SW38 ?, SW39 ?, SW4 ?, SW40 ?, SW41 ?, SW5 ?, SW6 ?, SW7 ?, SW8 ?, SW9 ?, U1 ?, U2 ?, U3 ?, U4 ?, U5 ?, U6 ?

Commit message: Place the board by writing the file, not through KiCad's API
place_keypad.py asks pcbnew to put footprints at absolute millimetre
positions. Under KiCad 10.0 that does not work: the first run put all 45
footprints it touched 414.5 mm from where it asked, a second run put them
345.0 mm out, and the board outline and comment rectangles drawn through the
same API in the same run landed exactly right. Reading a position back returns
the value that was asked for, so neither the script nor fix_offset.py could
tell that anything had gone wrong.

The relative geometry was never in question -- one clean translation of the
whole block, every rotation correct -- so this keeps the arithmetic and
changes only how it reaches the board.

tools/place_board.py rewrites the (at ...) lines in default.kicad_pcb from
outside KiCad. It needs no pcbnew and no conda environment, and its work shows
up in git diff: 119 changed lines, every one a position. The 74 parts step 7
still has to place by hand move as a block to the right of the board, keeping
their arrangement, rather than sitting 600 mm off the page.

The board file here is the corrected one: the 38 dome sites span board Y 62 to
134 inside the keyboard area, the six top-edge parts sit along the top edge,
and J2 is on the back at (9.00, 30.15).

Co-Authored-By: Claude Opus 5 (1M context) <noreply@anthropic.com>
Claude-Session: https://claude.ai/code/session_01QqQ2eJFoahQ6u3RFAgdwby
Parts:
- moved C14 974.6 mm to (103.0, 120.7)
- moved C16 974.6 mm to (117.3, 124.1)
- moved C18 974.6 mm to (96.9, 120.7)
- moved C5 974.6 mm to (156.8, 50.3)
- moved LS1 974.6 mm to (122.2, 36.0)
- moved R16 974.6 mm to (132.1, 49.7)
- moved R19 974.6 mm to (132.1, 45.7)
- moved TP7 974.6 mm to (171.9, 20.0)
- moved U4 974.6 mm to (123.7, 124.0)
- moved BT1 974.6 mm to (137.0, 119.5)
- moved C1 974.6 mm to (166.5, 37.5)
- moved C10 974.6 mm to (166.5, 42.0)
- moved C11 974.6 mm to (129.9, 122.5)
- moved C12 974.6 mm to (166.5, 33.0)
- moved C13 974.6 mm to (129.9, 118.0)
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
Commit message: Push the six top-edge parts out towards the case wall
Barnaby pointed out that the slider knob, the USB-C mouth and the rest need
to reach past the board edge to be usable through the case. They were not:
the USB-C mouth sat exactly on the outline and the slider knob 0.80 mm past
it, against 2.00 mm from the board edge to the case's outer surface (0.80 mm
of assembly clearance plus a 1.20 mm wall).

Each part is now as far out as its own pads allow, measured from the library
footprints rather than estimated:

  slider      2.30 mm past the edge, set to stand 0.3 mm proud of the case
  USB-C       1.20 mm, stopped by its through-hole shield legs
  status LED  1.12 mm
  IR emitter  1.08 mm
  tact x2     0.24 mm

Only the slider reaches the outside; the case has to come to the other five
with a recessed chamfered USB-C mouth, clear holes for the two LEDs and
pinholes for the recovery buttons.

The tact switches moved the other way, 1.50 to 1.80, because at 1.50 their
pads sat exactly on the board outline with no copper-to-edge clearance. That
was a fault, not a trade-off.

Also adds the two footprints for soldering the frontlight sliver to the main
board instead of wiring it: a castellated half-hole for the sliver's end edge
and the land it solders onto. Nothing uses them yet; the netlist change is a
separate step.

Co-Authored-By: Claude Opus 5 (1M context) <noreply@anthropic.com>
Claude-Session: https://claude.ai/code/session_01QqQ2eJFoahQ6u3RFAgdwby
Parts:
- moved SW39 1.50 mm to (11.0, 1.50)
- moved J1 1.20 mm to (36.0, 2.48)
- moved D5 0.75 mm to (48.0, 1.05)
- moved D4 0.70 mm to (22.0, 0.90)
- moved SW40 0.30 mm to (66.0, 1.80)
- moved SW41 0.30 mm to (57.0, 1.80)
Changed lines of the file:
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@@
 	(footprint "Button_Switch_SMD:SW_SPDT_CK_JS102011SAQN"
 		(layer "F.Cu")
-		(at 11 3 180)
+		(at 11 1.5 180)
 		(descr "Sub-miniature slide switch, right-angle, http://www.ckswitches.com/media/1422/js.pdf")
 		(tags "switch spdt")
@@
 	(footprint "hp42s:Vishay_VSMB2943SLX01_SideView"
 		(layer "F.Cu")
-		(at 22 1.6)
+		(at 22 0.9)
 		(descr "Vishay VSMB2943SLX01, 940 nm side-looking IR emitter, 2.3x2.55x2.3 mm. Pads per the IPC 7351 solder pad proposal in Vishay document 83479 rev 1.2. Lens faces -y; optical axis sits 1.2 mm above the board face the part is soldered to. Pad 1 = cathode.")
 		(tags "LED IR 940nm side-view sidelooker VSMB2943SLX01")
@@
 	(footprint "hp42s:Alps_SKRTLAE010_SidePush"
 		(layer "F.Cu")
-		(at 57 1.5 180)
+		(at 57 1.8 180)
 		(descr "Alps SKRTLAE010, 4.5x3.4x3.3 mm side-push tact switch with guide bosses. Land, both dia 0.9 boss holes and the prohibited copper area from the Alps TACT Switch catalogue page 250. Terminals 1 and 3 are commoned inside the switch, so both are pad 1. MP is the ground terminal. Plunger faces +y and stands 0.84 mm proud.")
 		(tags "tact switch side-push Alps SKRT SKRTLAE010")
@@
 	(footprint "Connector_USB:USB_C_Receptacle_GCT_USB4105-xx-A_16P_TopMnt_Horizontal"
 		(layer "F.Cu")
-		(at 36 3.675 180)
+		(at 36 2.475 180)
 		(descr "USB 2.0 Type C Receptacle, GCT, 16P, top mounted, horizontal, 5A: https://gct.co/files/drawings/usb4105.pdf")
 		(tags "USB C Type-C Receptacle SMD USB 2.0 16P 16C USB4105-15-A USB4105-15-A-060 USB4105-15-A-120 USB4105-GF-A USB4105-GF-A-060 USB4105-GF-A-120")
@@
 	(footprint "hp42s:Dialight_599_BiColor_1208_RA"
 		(layer "F.Cu")
-		(at 48 1.8)
+		(at 48 1.05)
 		(descr "Dialight 599 series MicroLED, bi-colour 1208 right angle, 3.0x2.0x1.0 mm. Pads per the recommended layout on page 1 of the Dialight datasheet. Lens faces -y; it spans roughly 1.0 to 2.0 mm above the board face the part is soldered to. Pad 2 = common anode, pad 3 = LED die 1, pad 1 = LED die 2.")
 		(tags "LED bicolor side-view right-angle Dialight 599 1208")
@@
 	(footprint "hp42s:Alps_SKRTLAE010_SidePush"
 		(layer "F.Cu")
-		(at 66 1.5 180)
+		(at 66 1.8 180)
 		(descr "Alps SKRTLAE010, 4.5x3.4x3.3 mm side-push tact switch with guide bosses. Land, both dia 0.9 boss holes and the prohibited copper area from the Alps TACT Switch catalogue page 250. Terminals 1 and 3 are commoned inside the switch, so both are pad 1. MP is the ground terminal. Plunger faces +y and stands 0.84 mm proud.")
 		(tags "tact switch side-push Alps SKRT SKRTLAE010")

Commit message: First pass at placing the remaining 74 parts
Everything now has a position: 56 footprints on the front, 63 on the back,
none overlapping, none crossing the outline, none in the battery bay or the
module's antenna keepout.

The battery bay is what shapes this. The cell on the back at the top leaves
the electronics the back below Y 59, plus two slivers of front that nothing
else wanted: Y 5-12 above the glass and Y 48.3-59 between the glass and the
keys. The USB front end goes in the first, behind its connector rather than
60 mm of unprotected D+/D- away from it; the frontlight sliver's two pads go
in the second.

On the back: the panel's boost top left near J2, the frontlight driver top
right and as far from both switchers as the board allows, the cell connector
below the bay, the power chain through the middle, and the module at the
bottom rotated 180 so its antenna radiates off the board edge into the chin,
which docs/front-face.md already keeps the faceplate out of.

place_board.py now sets layer as well as position; flipping a footprint is a
swap of every F.* layer name for its B.* twin, which is what KiCad itself did
to J2.

Reasoning and the four open questions are in docs/placement.md.

Co-Authored-By: Claude Opus 5 (1M context) <noreply@anthropic.com>
Claude-Session: https://claude.ai/code/session_01QqQ2eJFoahQ6u3RFAgdwby
Parts:
- BT1, C10, C11, C12, C13, C14, C15, C16, C17, C18, C19, C2, C20, C21, C22, C3, C4, C5, C6, C7, C8, C9, D1, D2, D3, D6, L1, L2, L3, LS1, Q1, R10, R11, R12, R13, R14, R15, R16, R17, R22, R23, R24, R3, R4, R5, R6, R7, R8, R9, TP10, TP11, TP4, TP5, TP6, TP7, TP8, TP9, U2, U3, U4, U5, U6: moved to B.Cu
- moved Q2 180.9 mm to (29.1, 9.60)
- moved R17 180.6 mm to (11.0, 119.0)
- moved C19 171.3 mm to (3.05, 68.2)
- moved R2 170.7 mm to (21.9, 9.60)
- moved Q1 164.0 mm to (8.85, 61.2)
- moved C10 157.1 mm to (11.2, 66.2)
- moved R1 156.3 mm to (19.1, 9.60)
- moved U1 153.6 mm to (15.6, 9.60)
- moved C12 153.1 mm to (17.1, 66.2)
- moved L2 150.8 mm to (4.35, 62.4)
- moved C3 149.7 mm to (23.1, 84.8)
- moved R20 149.0 mm to (38.5, 9.60)
- moved R15 148.1 mm to (27.1, 60.5)
- moved C2 146.8 mm to (19.8, 84.8)
- moved D1 146.5 mm to (13.2, 61.0)
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