File: elec/layout/default/default.kicad_pcb (KiCad board)
At the start: 4 copper layers, 76 x 155 mm, 118 parts, among them J1 ?, J2 ?, Q1 ?, Q2 ?, SW1 ?, SW10 ?, SW11 ?, SW12 ?, SW13 ?, SW14 ?, SW15 ?, SW16 ?, SW17 ?, SW18 ?, SW19 ?, SW2 ?, SW20 ?, SW21 ?, SW22 ?, SW23 ?, SW24 ?, SW25 ?, SW26 ?, SW27 ?, SW28 ?, SW29 ?, SW3 ?, SW30 ?, SW31 ?, SW32 ?, SW33 ?, SW34 ?, SW35 ?, SW36 ?, SW37 ?, SW38 ?, SW39 ?, SW4 ?, SW40 ?, SW5 ?, SW6 ?, SW7 ?, SW8 ?, SW9 ?, U1 ?, U2 ?, U3 ?, U4 ?, U5 ?, U6 ?

Commit message: Import the MIP netlist
Parts:
- removed the C11 at (7.62, 71.3)
- removed the C15 at (12.1, 73.9)
- removed the C17 at (20.3, 84.0)
- removed C18: ?, Capacitor_SMD:C_0805_2012Metric
- removed C19: ?, Capacitor_SMD:C_0603_1608Metric
- removed the D1 at (20.3, 80.8)
- removed the D2 at (6.35, 90.4)
- removed the D3 at (12.7, 90.4)
- removed the Q1 at (8.89, 82.1)
- added U6: ?, hp42s:TI_YFF0006_DSBGA-6_0.88x1.23mm_P0.4mm, F.Cu at (109.8, 144.6)
- added U7: ?, hp42s:MicroCrystal_C7_3.2x1.5mm_RV-8263, F.Cu at (110.7, 132.8)
- C10, C12, C13, R14: moved to F.Cu
- C14: footprint Capacitor_SMD:C_0603_1608Metric -> Capacitor_SMD:C_0402_1005Metric; moved to F.Cu
- J2: footprint Connector_FFC-FPC:Amphenol_F32Q-1A7x1-11024_1x24-1MP_P0.5mm_Horizontal -> hp42s:Hirose_FH34SRJ-10S-0.5SH_1x10-1MP_P0.50mm_Horizontal; moved to F.Cu
- L2: footprint Inductor_SMD:L_Bourns-SRN4018 -> Inductor_SMD:L_Murata_DFE201610P
- R15: footprint Resistor_SMD:R_0603_1608Metric -> Resistor_SMD:R_0402_1005Metric; moved to F.Cu
- moved J2 138.8 mm to (101.8, 132.3), turned to 0 degrees
- moved C14 122.5 mm to (104.9, 148.2)
- moved C13 121.8 mm to (105.5, 140.0)
- moved C10 121.0 mm to (99.5, 144.5)
- moved R15 120.2 mm to (111.0, 139.7)
- moved R14 118.0 mm to (105.0, 144.2)
- moved C12 111.2 mm to (99.5, 140.0)
- renumbered C16 to C11, C20 to C15, C21 to C16, C22 to C17, D4 to D1, D5 to D2, D6 to D3, Q2 to Q1, U6 to U8
Connections:
- net frontlight-sw renamed sw
- C10 pad 1: v3v3 -> v5
- C11 pad 1: v3v3 -> sys
- C12 pad 1: vsh1 -> v5
- C13 pad 1: vsh2 -> v5
- C14 pad 1: vsl -> v3v3
- J2 pad 1: nc1 -> mip_sck
- J2 pad 10: epd_rst -> gnd
- J2 pad 2: gdr -> mip_mosi
- J2 pad 3: rese -> mip_cs
- J2 pad 4: nc4 -> extcomin
- J2 pad 5: vsh2 -> mip_disp
- J2 pad 6: tscl -> v5
- J2 pad 7: tsda -> v5
- J2 pad 8: gnd -> v5
- J2 pad 9: epd_busy -> gnd
- L2 pad 1: v3v3 -> sys
- L2 pad 2: display-sw -> sw5
- R14 pad 1: gdr -> mip_pwr
- R15 pad 1: rese -> mip_clkoe
- U5 pad 28: epd_cs -> mip_cs
- U5 pad 29: epd_dc -> mip_disp
- U5 pad 31: epd_rst -> mip_pwr
- U5 pad 32: epd_busy -> mip_clkoe
- U5 pad 33: epd_sck -> mip_sck
- U5 pad 34: epd_mosi -> mip_mosi
Routing:
- net (no net): track 0.00 -> 535.9 mm, vias 0 -> 18
- net epd_rst: track 145.9 -> 0.00 mm, vias 12 -> 0
- net mip_pwr: track 0.00 -> 145.9 mm, vias 0 -> 12
- net mip_cs: track 0.00 -> 145.6 mm, vias 0 -> 12
- net epd_cs: track 145.6 -> 0.00 mm, vias 12 -> 0
- net epd_busy: track 144.2 -> 0.00 mm, vias 4 -> 0
- net mip_clkoe: track 0.00 -> 144.2 mm, vias 0 -> 4
- net mip_mosi: track 0.00 -> 141.2 mm, vias 0 -> 6
- net epd_mosi: track 141.2 -> 0.00 mm, vias 6 -> 0
- net epd_dc: track 140.6 -> 0.00 mm, vias 10 -> 0
- net mip_disp: track 0.00 -> 140.6 mm, vias 0 -> 10
- net epd_sck: track 138.3 -> 0.00 mm, vias 10 -> 0
- net mip_sck: track 0.00 -> 138.3 mm, vias 0 -> 10
- net rese: track 84.2 -> 0.00 mm, vias 4 -> 0
- net gdr: track 75.3 -> 0.00 mm, vias 2 -> 0
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