File: elec/layout/default/default.kicad_pcb (KiCad board)
At the start: 4 copper layers, 76 x 146 mm, 100 parts, among them J1 ?, J2 ?, Q1 ?, SW1 ?, SW10 ?, SW11 ?, SW12 ?, SW13 ?, SW14 ?, SW15 ?, SW16 ?, SW17 ?, SW18 ?, SW19 ?, SW2 ?, SW20 ?, SW21 ?, SW22 ?, SW23 ?, SW24 ?, SW25 ?, SW26 ?, SW27 ?, SW28 ?, SW29 ?, SW3 ?, SW30 ?, SW31 ?, SW32 ?, SW33 ?, SW34 ?, SW35 ?, SW36 ?, SW37 ?, SW38 ?, SW39 ?, SW4 ?, SW40 ?, SW5 ?, SW6 ?, SW7 ?, SW8 ?, SW9 ?, U1 ?, U2 ?, U3 ?, U4 ?, U5 ?, U6 ?, U7 ?

Commit message: mip: netlist import, WROOM + NAND
Parts:
- added C15: ?, Capacitor_SMD:C_0402_1005Metric, F.Cu at (98.3, 77.0)
- added R16: ?, Resistor_SMD:R_0402_1005Metric, F.Cu at (93.5, 77.0)
- added U8: ?, hp42s:SPI_NAND_UPDFN-8_8x6mm_P1.27mm, F.Cu at (97.3, 70.3)
- U5: footprint RF_Module:ESP32-S2-MINI-1 -> hp42s:ESP32-S3-WROOM-1
- renumbered R16 to R17, R17 to R18, R18 to R19, R19 to R20, R20 to R21, R24 to R22, TP3 to TP1, TP4 to TP2, TP5 to TP3, TP6 to TP4, TP7 to TP5, TP8 to TP6, TP9 to TP7, TP10 to TP8, TP11 to TP9
Connections:
- U5 pad 10: col4 -> i2c_sda
- U5 pad 11: col5 -> i2c_scl
- U5 pad 13: row1 -> usb_dm
- U5 pad 14: row2 -> usb_dp
- U5 pad 15: row3 -> io3
- U5 pad 16: row4 -> io46
- U5 pad 17: row5 -> row1
- U5 pad 18: row6 -> row2
- U5 pad 19: chg_stat2 -> row3
- U5 pad 2: gnd -> v3v3
- U5 pad 20: led_red -> row4
- U5 pad 21: i2c_sda -> row5
- U5 pad 22: i2c_scl -> row6
- U5 pad 23: usb_dm -> buzzer
- U5 pad 24: usb_dp -> ir_led
- U5 pad 25: buzzer -> chg_stat
- U5 pad 26: (no net) -> mip_disp
- U5 pad 27: ir_led -> boot
- U5 pad 28: mip_cs -> mip_pwr
- U5 pad 29: mip_disp -> mip_clkoe
- U5 pad 3: v3v3 -> en
- U5 pad 30: chg_stat -> mip_sck
- U5 pad 31: mip_pwr -> mip_mosi
- U5 pad 32: mip_clkoe -> led_green
- U5 pad 33: mip_sck -> mip_cs
- U5 pad 34: mip_mosi -> flash_cs
- U5 pad 35: led_green -> flash_miso
- U5 pad 36: io40 -> uart0_rx
- U5 pad 37: frontlight_pwm -> uart0_tx
- U5 pad 38: (no net) -> col1
- U5 pad 39: uart0_tx -> col0
- U5 pad 4: boot -> col2
- U5 pad 40: uart0_rx -> gnd
- U5 pad 41: (no net) -> gnd
- U5 pad 5: col0 -> col3
- U5 pad 6: col1 -> col4
- U5 pad 7: (no net) -> col5
- U5 pad 8: col2 -> chg_stat2
- U5 pad 9: col3 -> led_red
